Commit message: modified the mass

File: urdf/delto.urdf (robot description, URDF)
Before this commit: robot delto, 13 links, 12 joints
Links:
- link base_link: mass 0.32613215710018 -> 0.292
- link finger1_link1: mass 0.32613215710018 -> 0.048
- link finger1_link2: mass 0.32613215710018 -> 0.012
- link finger1_link3: mass 0.32613215710018 -> 0.038
- link finger1_link4: mass 0.32613215710018 -> 0.06
- link finger2_link1: mass 0.32613215710018 -> 0.048
- link finger2_link2: mass 0.32613215710018 -> 0.012
- link finger2_link3: mass 0.32613215710018 -> 0.038
- link finger2_link4: mass 0.32613215710018 -> 0.06
- link finger3_link1: mass 0.32613215710018 -> 0.048
- link finger3_link2: mass 0.32613215710018 -> 0.012
- link finger3_link3: mass 0.32613215710018 -> 0.038
- link finger3_link4: mass 0.32613215710018 -> 0.06

File: urdf/delto.xacro (robot description, xacro)
@@ -26,5 +26,5 @@
         rpy="0 0 0" />
       <mass
-        value="0.32613215710018" />
+        value="0.292" />
       <inertia
         ixx="0"
@@ -66,5 +66,5 @@
         rpy="0 0 0" />
       <mass
-        value="0.32613215710018" />
+        value="0.048" />
       <inertia
         ixx="0"
@@ -135,5 +135,5 @@
         rpy="0 0 0" />
       <mass
-        value="0.32613215710018" />
+        value="0.012" />
       <inertia
         ixx="0"
@@ -204,5 +204,5 @@
         rpy="0 0 0" />
       <mass
-        value="0.32613215710018" />
+        value="0.038" />
       <inertia
         ixx="0"
@@ -273,5 +273,5 @@
         rpy="0 0 0" />
       <mass
-        value="0.32613215710018" />
+        value="0.06" />
       <inertia
         ixx="0"
@@ -342,5 +342,5 @@
         rpy="0 0 0" />
       <mass
-        value="0.32613215710018" />
+        value="0.048" />
       <inertia
         ixx="0"
@@ -411,5 +411,5 @@
         rpy="0 0 0" />
       <mass
-        value="0.32613215710018" />
+        value="0.012" />
       <inertia
         ixx="0"
@@ -480,5 +480,5 @@
         rpy="0 0 0" />
       <mass
-        value="0.32613215710018" />
+        value="0.038" />
       <inertia
         ixx="0"
@@ -549,5 +549,5 @@
         rpy="0 0 0" />
       <mass
-        value="0.32613215710018" />
+        value="0.06" />
       <inertia
         ixx="0"
@@ -618,5 +618,5 @@
         rpy="0 0 0" />
       <mass
-        value="0.32613215710018" />
+        value="0.048" />
       <inertia
         ixx="0"
@@ -687,5 +687,5 @@
         rpy="0 0 0" />
       <mass
-        value="0.32613215710018" />
+        value="0.012" />
       <inertia
         ixx="0"
@@ -756,5 +756,5 @@
         rpy="0 0 0" />
       <mass
-        value="0.32613215710018" />
+        value="0.038" />
       <inertia
         ixx="0"
@@ -825,5 +825,5 @@
         rpy="0 0 0" />
       <mass
-        value="0.32613215710018" />
+        value="0.06" />
       <inertia
         ixx="0"
